File: osukeypad-pcb.kicad_pcb (KiCad board)
At the start: 2 copper layers, 93.7 x 38.1 mm, 24 parts, among them SW1 SW_Push, U1 ATmega32U4-AU, Y1 16MHz

Commit message: osukeypad-update-2
Parts:
- moved C3 1.15 mm to (32.9, 75.7)
- moved C5 0.90 mm to (62.1, 57.8)
- moved D1 0.79 mm to (101.6, 61.9)
- moved D3 0.79 mm to (120.7, 61.8)
- moved D4 0.79 mm to (120.7, 80.9)
- moved C4 0.38 mm to (70.2, 58.0)
Routing:
- net +5V: track 133.1 -> 0.36 mm
- net GND: track 133.3 -> 2.19 mm
- net ROW0: track 20.9 -> 0.00 mm
- net ROW1: track 20.6 -> 0.15 mm
- net COL0: track 19.1 -> 0.01 mm
- net COL1: track 19.1 -> 0.01 mm
- net Net-(C5-Pad1): track 17.6 -> 0.82 mm
- net VCC: track 16.3 -> 2.84 mm
- net Net-(R3-Pad2): track 10.1 -> 0.15 mm
- net Net-(C4-Pad1): track 12.3 -> 2.39 mm
- net Net-(D2-Pad2): track 8.86 -> 0.82 mm
- net Net-(D4-Pad2): track 8.07 -> 0.82 mm
- net Net-(D3-Pad2): track 8.07 -> 0.82 mm
- net Net-(D1-Pad2): track 8.07 -> 0.82 mm
- net Net-(R4-Pad2): track 4.82 -> 0.00 mm
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Other:
- net class Default: trace_width 0.4 -> 0.25
- net class Power: trace_width 0.4 -> 0.25

Commit message: osupad-update-3
Parts:
- moved C3 43.9 mm to (76.1, 67.5), turned to 90 degrees
- moved C1 20.8 mm to (57.4, 62.2)
- moved R3 18.1 mm to (54.2, 62.0)
- moved C7 10.4 mm to (56.8, 72.4), turned to 180 degrees
- moved SW1 9.84 mm to (45.3, 81.5)
- moved F1 6.51 mm to (39.0, 71.0)
- moved C2 5.43 mm to (55.8, 77.8), turned to 270 degrees
- moved R4 1.96 mm to (78.4, 79.2)
- moved R2 1.10 mm to (46.2, 64.4)
- moved R1 1.08 mm to (42.9, 64.4)
- moved C4 0.26 mm to (70.0, 58.0)
- moved USB1 0.18 mm to (45.0, 54.1)
- moved C5 0.13 mm to (62.2, 57.8)
Routing:
- net GND: track 2.19 -> 151.4 mm
- net +5V: track 0.36 -> 126.4 mm, vias 0 -> 5
- net COL1: track 0.01 -> 58.0 mm
- net ROW1: track 0.15 -> 57.6 mm
- net COL0: track 0.01 -> 38.6 mm
- net Net-(R3-Pad2): track 0.15 -> 33.0 mm, vias 0 -> 2
- net ROW0: track 0.00 -> 20.4 mm
- net Net-(C5-Pad1): track 0.82 -> 15.2 mm
- net VCC: track 2.84 -> 12.8 mm
- net Net-(C4-Pad1): track 2.39 -> 11.9 mm
- net Net-(R4-Pad2): track 0.00 -> 6.96 mm
- net Net-(D2-Pad2): track 0.82 -> 7.61 mm
- net Net-(D4-Pad2): track 0.82 -> 7.61 mm
- net Net-(D3-Pad2): track 0.82 -> 7.61 mm
- net Net-(D1-Pad2): track 0.82 -> 7.41 mm
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- added copper zone on B.Cu, net GND
Other:
- board size 93.7 x 38.1 mm -> 86.1 x 38.2 mm
- net class Power: trace_width 0.25 -> 0.4

Commit message: osukeypad-update-4
Routing:
- removed copper zone on B.Cu, net GND
Changed lines of the file:
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@@
   (gr_arc (start 38.481 54.70525) (end 38.481 52.324) (angle -90) (layer Edge.Cuts) (width 0.12))
   (gr_arc (start 119.85625 54.76875) (end 122.2375 54.76875) (angle -90) (layer Edge.Cuts) (width 0.12))
-  (via (at 50.673 79.629) (size 0.8) (drill 0.4) (layers F.Cu B.Cu) (net 19))
-  (via (at 77.978 68.453) (size 0.4) (drill 0.3) (layers F.Cu B.Cu) (net 2))
-  (via (at 75.311 81.788) (size 0.8) (drill 0.4) (layers F.Cu B.Cu) (net 2))
-  (via (at 59.055 76.2) (size 0.4) (drill 0.3) (layers F.Cu B.Cu) (net 2))
-  (via (at 59.055 71.12) (size 0.8) (drill 0.4) (layers F.Cu B.Cu) (net 2))
-  (via (at 55.753 61.468) (size 0.8) (drill 0.4) (layers F.Cu B.Cu) (net 2))
-  (via (at 52.451 62.992) (size 0.8) (drill 0.4) (layers F.Cu B.Cu) (net 19))
   (segment (start 67.36875 57.0375) (end 67.46875 57.0375) (width 0.4) (layer B.Cu) (net 1))
   (segment (start 65.448748 58.7375) (end 65.26875 58.7375) (width 0.4) (layer B.Cu) (net 1))
@@
   (segment (start 64.93125 68.245002) (end 66.53125 69.845002) (width 0.4) (layer B.Cu) (net 1))
   (segment (start 64.93125 67.3) (end 64.93125 68.245002) (width 0.4) (layer B.Cu) (net 1))
+  (via (at 77.978 68.453) (size 0.4) (drill 0.3) (layers F.Cu B.Cu) (net 2))
+  (via (at 75.311 81.788) (size 0.8) (drill 0.4) (layers F.Cu B.Cu) (net 2))
+  (via (at 59.055 76.2) (size 0.4) (drill 0.3) (layers F.Cu B.Cu) (net 2))
+  (via (at 59.055 71.12) (size 0.8) (drill 0.4) (layers F.Cu B.Cu) (net 2))
+  (via (at 55.753 61.468) (size 0.8) (drill 0.4) (layers F.Cu B.Cu) (net 2))
   (segment (start 71.20625 78.7) (end 70.53125 78.7) (width 0.4) (layer B.Cu) (net 2))
   (segment (start 73.406263 80.900013) (end 71.20625 78.7) (width 0.4) (layer B.Cu) (net 2))
@@
   (segment (start 45.898 74.6) (end 60.83125 74.6) (width 0.25) (layer B.Cu) (net 18))
   (segment (start 44.850509 73.552509) (end 45.898 74.6) (width 0.25) (layer B.Cu) (net 18))
+  (via (at 50.673 79.629) (size 0.8) (drill 0.4) (layers F.Cu B.Cu) (net 19))
+  (via (at 52.451 62.992) (size 0.8) (drill 0.4) (layers F.Cu B.Cu) (net 19))
   (segment (start 52.481 62.962) (end 52.451 62.992) (width 0.25) (layer B.Cu) (net 19))
   (segment (start 54.229 62.962) (end 52.481 62.962) (width 0.25) (layer B.Cu) (net 19))
@@
   (segment (start 78.359 78.262) (end 72.96825 78.262) (width 0.25) (layer B.Cu) (net 20))
   (segment (start 60.83125 69.8) (end 61.137 69.8) (width 0.4) (layer B.Cu) (net 40))
-  (zone (net 1) (net_name GND) (layer B.Cu) (hatch edge 0.508)
-    (connect_pads (clearance 0.508))
-    (min_thickness 0.254)
-    (fill yes (arc_segments 32) (thermal_gap 0.508) (thermal_bridge_width 0.508))
-    (polygon
-      (pts
-        (xy 36.83 53.34) (xy 83.82 53.34) (xy 83.82 90.17) (xy 37.211 89.916)
-      )
-    )
-  )
 )

Commit message: osukeypad-update-4
Parts:
- moved C2 7.60 mm to (62.5, 81.2)
- moved C4 7.37 mm to (77.3, 57.7)
- moved Y1 6.73 mm to (72.9, 57.7)
- moved F1 6.62 mm to (45.6, 70.5)
- moved USB1 6.61 mm to (51.6, 53.8)
- moved R2 6.55 mm to (52.8, 64.8)
- moved R1 6.49 mm to (49.4, 64.8)
- moved C1 6.39 mm to (63.8, 61.4)
- moved C5 6.35 mm to (68.6, 57.7)
- moved R3 6.25 mm to (60.5, 61.4)
- moved SW1 6.01 mm to (51.1, 83.1)
- moved U1 5.49 mm to (71.9, 72.1), turned to 45 degrees
- moved C7 5.11 mm to (60.9, 75.5)
- moved C3 5.01 mm to (80.5, 65.2)
- moved C6 3.47 mm to (72.3, 85.2)
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Routing:
- net GND: track 151.4 -> 223.2 mm
- net Net-(USB1-Pad6): track 0.00 -> 25.5 mm
- net +5V: track 126.4 -> 133.3 mm
- net Net-(R1-Pad1): track 26.1 -> 30.3 mm
- net Net-(C4-Pad1): track 11.9 -> 16.0 mm
- net Net-(C7-Pad1): track 3.33 -> 7.08 mm
- net Net-(R2-Pad1): track 25.2 -> 28.7 mm
- net ROW1: track 57.6 -> 55.5 mm
- net Net-(R4-Pad2): track 6.96 -> 8.86 mm
- net Net-(C5-Pad1): track 15.2 -> 17.1 mm
- net COL0: track 38.6 -> 36.9 mm
- net Net-(R3-Pad2): track 33.0 -> 34.3 mm
- net COL1: track 58.0 -> 56.8 mm, vias 1 -> 0
- net VCC: track 12.8 -> 12.3 mm
- added copper zone on B.Cu, net GND
Other:
- board size 86.1 x 38.2 mm -> 82.5 x 39.4 mm
- net class Default: via_dia 0.4 -> 0.8; via_drill 0.3 -> 0.4
- net class Power: trace_width 0.4 -> 0.3; via_dia 0.4 -> 0.8; via_drill 0.3 -> 0.4

Commit message: osukeypad-update-5
Other:
- board text added: "Peu Peex"
Changed lines of the file:
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@@
   (general
     (thickness 1.6)
-    (drawings 4)
+    (drawings 5)
     (tracks 233)
     (zones 0)
@@
     )
   )
+  (gr_text "Peu Peex" (at 60.325 88.10625) (layer F.SilkS)
+    (effects (font (size 1 1) (thickness 0.15)))
+  )
   (gr_line (start 40.64 91.44) (end 40.64 52.07) (layer Edge.Cuts) (width 0.05))
   (gr_line (start 123.19 91.44) (end 40.64 91.44) (layer Edge.Cuts) (width 0.05))
   (gr_line (start 123.19 52.07) (end 123.19 91.44) (layer Edge.Cuts) (width 0.05))
   (gr_line (start 123.19 52.07) (end 40.64 52.07) (layer Edge.Cuts) (width 0.05))
-  (via (at 65.405 76.2) (size 0.8) (drill 0.4) (layers F.Cu B.Cu) (net 2))
-  (via (at 74.93 85.09) (size 0.8) (drill 0.4) (layers F.Cu B.Cu) (net 2))
-  (via (at 58.42 62.357) (size 0.8) (drill 0.4) (layers F.Cu B.Cu) (net 19))
-  (via (at 56.8452 81.1276) (size 0.8) (drill 0.4) (layers F.Cu B.Cu) (net 19))
   (segment (start 60.20731 79.79881) (end 62.5475 82.139) (width 0.3) (layer B.Cu) (net 1))
   (segment (start 46.7655 84.9165) (end 45.9232 84.0742) (width 0.3) (layer B.Cu) (net 1))
@@
   (segment (start 44.36799 77.38799) (end 44.36799 71.264464) (width 0.3) (layer B.Cu) (net 1))
   (segment (start 46.77881 79.79881) (end 44.36799 77.38799) (width 0.3) (layer B.Cu) (net 1))
+  (via (at 65.405 76.2) (size 0.8) (drill 0.4) (layers F.Cu B.Cu) (net 2))
+  (via (at 74.93 85.09) (size 0.8) (drill 0.4) (layers F.Cu B.Cu) (net 2))
   (segment (start 62.5475 79.3623) (end 62.5475 80.264) (width 0.3) (layer B.Cu) (net 2))
   (segment (start 62.484 79.2988) (end 62.5475 79.3623) (width 0.3) (layer B.Cu) (net 2))
@@
   (segment (start 53.84081 77.5376) (end 54.254305 77.951095) (width 0.25) (layer B.Cu) (net 18))
   (segment (start 54.254305 77.951095) (end 68.329647 77.951095) (width 0.25) (layer B.Cu) (net 18))
+  (via (at 58.42 62.357) (size 0.8) (drill 0.4) (layers F.Cu B.Cu) (net 19))
+  (via (at 56.8452 81.1276) (size 0.8) (drill 0.4) (layers F.Cu B.Cu) (net 19))
   (segment (start 56.7563 81.2165) (end 56.8452 81.1276) (width 0.25) (layer B.Cu) (net 19))
   (segment (start 54.1655 81.2165) (end 56.7563 81.2165) (width 0.25) (layer B.Cu) (net 19))
