File: osukeypad-pcb.kicad_pcb (KiCad board)
At the start: 2 copper layers, 82.5 x 39.4 mm, 24 parts, among them SW1 SW_Push, U1 ATmega32U4-AU, Y1 16MHz

Commit message: osukeypad-update-8
Routing:
- net Net-(USB1-Pad6): track 25.5 -> 1.00 mm
Changed lines of the file:
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@@
     (thickness 1.6)
     (drawings 5)
-    (tracks 233)
+    (tracks 225)
     (zones 0)
     (modules 24)
@@
       (drillshape 0)
       (scaleselection 1)
-      (outputdirectory "../../../Área de Trabalho/"))
+      (outputdirectory "PCB/"))
   )
   (net 0 "")
@@
   (segment (start 80.899 72.964982) (end 78.804436 70.870418) (width 0.25) (layer B.Cu) (net 20))
   (segment (start 80.899 78.486) (end 80.899 72.964982) (width 0.25) (layer B.Cu) (net 20))
-  (segment (start 49.012 53.848) (end 55.212 53.848) (width 0.25) (layer B.Cu) (net 44))
-  (segment (start 47.912 53.848) (end 49.012 53.848) (width 0.25) (layer B.Cu) (net 44))
-  (segment (start 47.912 53.848) (end 47.912 58.348) (width 0.25) (layer B.Cu) (net 44))
   (segment (start 55.212 57.848) (end 55.212 58.348) (width 0.25) (layer B.Cu) (net 44))
-  (segment (start 54.112 56.748) (end 55.212 57.848) (width 0.25) (layer B.Cu) (net 44))
-  (segment (start 49.012 56.748) (end 54.112 56.748) (width 0.25) (layer B.Cu) (net 44))
-  (segment (start 47.912 57.848) (end 49.012 56.748) (width 0.25) (layer B.Cu) (net 44))
   (segment (start 47.912 58.348) (end 47.912 57.848) (width 0.25) (layer B.Cu) (net 44))
-  (segment (start 55.212 55.448) (end 55.212 58.348) (width 0.25) (layer B.Cu) (net 44))
-  (segment (start 55.212 53.848) (end 55.212 55.448) (width 0.25) (layer B.Cu) (net 44))
   (zone (net 1) (net_name GND) (layer B.Cu) (hatch edge 0.508)
     (connect_pads (clearance 0.508))
@@
     (polygon
       (pts
-        (xy 40.64 52.07) (xy 84.074 52.07) (xy 83.82 91.44) (xy 40.64 91.44)
+        (xy 41.275 52.3875) (xy 84.1375 52.3875) (xy 84.1375 91.28125) (xy 41.275 91.28125)
       )
     )
